File: STM32_HID_controller_shoulder/STM32_HID_controller-right.kicad_pcb (KiCad board)
At the start: 2 copper layers, 25 x 56 mm, 5 parts, among them J4 Conn_01x03_Socket

Commit message: changed shoulder to right orientation
Connections:
- J4 pad 1: Net-(J4-Pin_1) -> GND
- J4 pad 3: GND -> Net-(J4-Pin_3)
- trigger1 pad 2: Net-(J4-Pin_1) -> Net-(J4-Pin_3)
Routing:
- net Net-(J4-Pin_3): track 0.00 -> 38.8 mm
- net Net-(J4-Pin_1): track 38.1 -> 0.00 mm
Changed lines of the file:
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@@
 	(net 0 "")
 	(net 1 "GND")
-	(net 2 "Net-(J4-Pin_1)")
+	(net 2 "Net-(J4-Pin_3)")
 	(net 3 "Net-(J4-Pin_2)")
 	(footprint "Button_Switch_THT:SW_DIP_SPSTx01_Piano_10.8x4.1mm_W7.62mm_P2.54mm"
@@
 			(layers "*.Cu" "*.Mask")
 			(remove_unused_layers no)
-			(net 2 "Net-(J4-Pin_1)")
+			(net 2 "Net-(J4-Pin_3)")
 			(pinfunction "2")
 			(pintype "passive")
@@
 			(remove_unused_layers no)
 			(roundrect_rratio 0.147059)
-			(net 2 "Net-(J4-Pin_1)")
+			(net 1 "GND")
 			(pinfunction "Pin_1")
 			(pintype "passive")
@@
 			(layers "*.Cu" "*.Mask")
 			(remove_unused_layers no)
-			(net 1 "GND")
+			(net 2 "Net-(J4-Pin_3)")
 			(pinfunction "Pin_3")
 			(pintype "passive")
@@
 	)
 	(segment
-		(start 135 140)
-		(end 135 141.95)
+		(start 130 140)
+		(end 130 141.9)
 		(width 0.5)
 		(layer "F.Cu")
@@
 	)
 	(via
-		(at 135 141.95)
+		(at 130 141.9)
 		(size 0.7)
 		(drill 0.3)
@@
 	)
 	(segment
-		(start 124.05 145.95)
-		(end 124.05 164.43)
+		(start 135 140)
+		(end 141.251 146.251)
 		(width 0.3)
 		(layer "F.Cu")
@@
 	)
 	(segment
-		(start 130 140)
-		(end 124.05 145.95)
+		(start 141.251 146.251)
+		(end 141.251 163.129)
 		(width 0.3)
 		(layer "F.Cu")
@@
 	)
 	(segment
-		(start 124.05 164.43)
+		(start 141.251 163.129)
 		(end 132 172.38)
 		(width 0.3)
@@
 	)
 	(segment
+		(start 132.5 148.5)
+		(end 126 155)
+		(width 0.3)
+		(layer "F.Cu")
+		(net 3)
+	)
+	(segment
 		(start 132.5 140)
-		(end 132.5 149)
+		(end 132.5 148.5)
 		(width 0.3)
 		(layer "F.Cu")
-		(net 3)
-	)
-	(segment
-		(start 132.5 149)
-		(end 138.5 155)
-		(width 0.3)
-		(layer "F.Cu")
