File: STM32_HID_controller/STM32_HID_controller.kicad_sch (KiCad schematic)
At the start: 57 parts, among them J1 USB_B_Micro, J2 Conn_01x04_Pin, J3 Conn_01x03_Pin, J5 Conn_01x03_Pin, SW1 SW_SPDT, SW10 SW_Push, SW11 SW_Push, SW14 SW_Push, SW2 SW_Push, SW3 SW_Push, SW6 SW_Push, SW7 SW_Push, SW8 SW_Push, SW9 SW_Push, U1 STM32F446RETx, U2 AMS1117-3.3, U4 joystick_right, U5 joystick_left, U7 MPU-6050, Y1 8MHz

Commit message: Switch prototype completed
Parts:
- removed C19: 2.2n, Capacitor_SMD:C_0402_1005Metric, symbol Device:C
- removed C20: .1u, Capacitor_SMD:C_0402_1005Metric, symbol Device:C
- removed U2: AMS1117-3.3, Package_TO_SOT_SMD:SOT-223-3_TabPin2, symbol Regulator_Linear:AMS1117-3.3
- removed U7: MPU-6050, Sensor_Motion:InvenSense_QFN-24_4x4mm_P0.5mm, symbol Sensor_Motion:MPU-6050
- added C24: 2.2u, Capacitor_SMD:C_0201_0603Metric, symbol Device:C
- added U2: TLV1117-33, Package_TO_SOT_SMD:SOT-223-3_TabPin2, symbol Regulator_Linear:TLV1117-33
- added U3: USBLC6-2SC6, Package_TO_SOT_SMD:SOT-23-6, symbol Power_Protection:USBLC6-2SC6
- added U7: ICM-42670-P, ICM-42670-P:LGA14_2.5X3X0.76_IVS-M, symbol ICM-42670-P:ICM-42670-P
- C1, C10, C2, C22, C3, C4, C5, C7: MANUFACTURER (none) -> Murata Electronics; MPN (none) -> GRM155R71C104KA88D
- C11, C12: MANUFACTURER (none) -> Murata Electronics; MPN (none) -> GRM1555C1H100JA01D
- C13: MANUFACTURER (none) -> KEMET; MPN (none) -> C0805C226M8PACTU
- C14: MANUFACTURER (none) -> KEMET; MPN (none) -> C0805C106M8PACTU
- C15, C16, C17, C18, C23: MANUFACTURER (none) -> Murata Electronics; MPN (none) -> GRM155R71C103KA01D
- C21: footprint Capacitor_SMD:C_0402_1005Metric -> Capacitor_SMD:C_0603_1608Metric; MANUFACTURER (none) -> KEMET; MPN (none) -> C0603C475K8PACTU
- C6: MANUFACTURER (none) -> TDK; MPN (none) -> C1608X5R1A106K080AC
- C8, C9: MANUFACTURER (none) -> YAGEO; MPN (none) -> CC0402KRX5R6BB105
- D1: MANUFACTURER (none) -> Lite-On; MPN (none) -> LTST-C190KRKT
- FB1: MANUFACTURER (none) -> Murata Electronics; MPN (none) -> BLM18AG121SN1D
- J1: MANUFACTURER (none) -> Würth Elektronik; MPN (none) -> 629105150521
- J2: MANUFACTURER (none) -> Würth Elektronik; MPN (none) -> 61300411121
- J3, J5: MANUFACTURER (none) -> JST; MPN (none) -> S3B-EH(LF)(SN)
- R1: MANUFACTURER (none) -> YAGEO; MPN (none) -> RC0402FR-0710KL
- R2: MANUFACTURER (none) -> YAGEO; MPN (none) -> RC0402FR-071K5L
- R3, R4: MANUFACTURER (none) -> YAGEO; MPN (none) -> RC0402FR-074K7L
- SW1: MANUFACTURER (none) -> C&K / Littelfuse; MPN (none) -> PCM12SMTR
- SW10, SW11, SW14, SW2, SW3: MANUFACTURER (none) -> Omron Electronics Components; MPN (none) -> B3F-1000
- SW6, SW7, SW8, SW9: MANUFACTURER (none) -> Würth Elektronik; MPN (none) -> 430476085716
- U1: MANUFACTURER (none) -> STMicroelectronics; MPN (none) -> STM32F446RET6
- U4, U5: MPN (none) -> COM-09032
- Y1: MANUFACTURER (none) -> Jauch Quartz; MPN (none) -> J32SMX-H-F-G-I-8M0; Manufacturer (none) -> Jauch Quartz; private KLC_S4.1 -> KLC_S3.3
Connections:
- net +3.3V: now also C24.1, U2.2 (VO), U7.12 (AP_CS), U7.5 (VDDIO), U7.8 (VDD)
- net GND: now also J1.6 (Shield), C24.2, U2.1 (GND), U3.2 (GND), U7.1 (AP_SDO/AP_AD0), U7.6 (GND), U7.7 (FSYNC)
- net USB_D+: now also U3.1 (I/O1); no longer J1.3 (D+)
- net USB_D-: now also U3.3 (I/O2); no longer J1.2 (D-)
- net VBUS: now also U2.3 (VI), U3.5 (VBUS)
- net i2c_scl: now also U7.13 (AP_SCL/AP_SCLK)
- net i2c_sda: now also U7.14 (AP_SDA/AP_SDIO/AP_SDI)
- new net USB_J1_D+: J1.3 (D+), U3.6 (I/O1)
- new net USB_J1_D-: J1.2 (D-), U3.4 (I/O2)
- no-connect marks 28 -> 26
Other:
- moved on the sheet: C22, C23, R3, R4
